File: Badge_RP2350_FPGA/Badge_RP2350_FPGA.kicad_sch (KiCad schematic)
At the start: 0 parts

Commit message: fixes
Other:
- sheet GW1NR 9K FPGA renamed GW1N 9K FPGA
Changed lines of the file:
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@@
 		(title "RISC-V Summit Europe Badge")
 		(date "2026-03-29")
-		(rev "v1.53")
+		(rev "v1.54")
 		(company "SemiTO-V, RISC-V Student Team")
 		(comment 3 "License: CERN-OHL-W-2.0")
@@
 			(color 0 0 0 0)
 		)
-		(property "Sheetname" "GW1NR 9K FPGA"
+		(property "Sheetname" "GW1N 9K FPGA"
 			(at 236.22 88.1884 0)
 			(show_name no)
